Commit message: increase height of velodyne xacro

File: velodyne_description/urdf/example.urdf.xacro (robot description, xacro)
@@ -30,9 +30,9 @@
   <xacro:include filename="$(find velodyne_description)/urdf/VLP-16.urdf.xacro"/>
   <VLP-16 parent="base_link" name="velodyne" topic="/velodyne_points" hz="10" samples="440">
-    <origin xyz="0 0 0.4" rpy="0 0 0" />
+    <origin xyz="0 0 1.4" rpy="0 0 0" />
   </VLP-16>
   <xacro:include filename="$(find velodyne_description)/urdf/HDL-32E.urdf.xacro"/>
   <HDL-32E parent="base_link" name="velodyne2" topic="/velodyne_points2" hz="10" samples="220">
-    <origin xyz="0 0 0.6" rpy="0 0 0" />
+    <origin xyz="0 0 1.6" rpy="0 0 0" />
   </HDL-32E>
 </robot>
